Commit message: The overshooting of the mocdel was due to extremely small value of inertials. Increasing them to a realistic value fixed the issue

File: install/simple_four_wheels_description/share/simple_four_wheels_description/urdf/simple_four_wheels.xacro (robot description, xacro)
@@ -8,5 +8,5 @@
     <origin xyz="0.00014946656090056147 0.0 0.0025099644374021166" rpy="0 0 0"/>
     <mass value="0.4726809767637952"/>
-    <inertia ixx="0.000396" iyy="0.00057" izz="0.000963" ixy="0.0" iyz="0.0" ixz="-0.0"/>
+    <inertia ixx="0.0396" iyy="0.057" izz="0.0963" ixy="0.0" iyz="0.0" ixz="-0.0"/>
   </inertial>
   <visual>
@@ -28,5 +28,5 @@
     <origin xyz="-6.705522526129215e-10 0.0024999999999999883 3.7252904754037086e-11" rpy="0 0 0"/>
     <mass value="0.012330751165339937"/>
-    <inertia ixx="0.0" iyy="1e-06" izz="0.0" ixy="0.0" iyz="-0.0" ixz="0.0"/>
+    <inertia ixx="0.0" iyy="0.001" izz="0.0" ixy="0.0" iyz="-0.0" ixz="0.0"/>
   </inertial>
   <visual>
@@ -48,5 +48,5 @@
     <origin xyz="6.705522526129215e-10 -0.0024999999999999883 3.7252904754037086e-11" rpy="0 0 0"/>
     <mass value="0.012330751165339937"/>
-    <inertia ixx="0.0" iyy="1e-06" izz="0.0" ixy="0.0" iyz="-0.0" ixz="0.0"/>
+    <inertia ixx="0.0" iyy="0.001" izz="0.0" ixy="0.0" iyz="-0.0" ixz="0.0"/>
   </inertial>
   <visual>
@@ -68,5 +68,5 @@
     <origin xyz="-6.705522526129215e-10 -0.0024999999999999883 3.7252904754037086e-11" rpy="0 0 0"/>
     <mass value="0.012330751165339937"/>
-    <inertia ixx="0.0" iyy="1e-06" izz="0.0" ixy="-0.0" iyz="-0.0" ixz="0.0"/>
+    <inertia ixx="0.0" iyy="0.001" izz="0.0" ixy="0.0" iyz="0.0" ixz="0.0"/>
   </inertial>
   <visual>
@@ -88,5 +88,5 @@
     <origin xyz="6.705522456740276e-10 0.0024999999999999883 3.725291169293099e-11" rpy="0 0 0"/>
     <mass value="0.012330751165339937"/>
-    <inertia ixx="0.0" iyy="1e-06" izz="0.0" ixy="-0.0" iyz="-0.0" ixz="-0.0"/>
+    <inertia ixx="0.0" iyy="0.001" izz="0.0" ixy="0.0" iyz="0.0" ixz="0.0"/>
   </inertial>
   <visual>
@@ -108,5 +108,5 @@
     <origin xyz="2.675393073642285e-05 -1.8066378496689461e-07 0.00752491787548288" rpy="0 0 0"/>
     <mass value="0.01775564430500639"/>
-    <inertia ixx="1e-06" iyy="0.0" izz="0.0" ixy="0.0" iyz="0.0" ixz="-0.0"/>
+    <inertia ixx="0.001" iyy="0.0" izz="0.0" ixy="0.0" iyz="0.0" ixz="0.0"/>
   </inertial>
   <visual>
@@ -128,5 +128,5 @@
     <origin xyz="2.6753930736402032e-05 1.8066378496689461e-07 0.007524917875482751" rpy="0 0 0"/>
     <mass value="0.01775564430500639"/>
-    <inertia ixx="1e-06" iyy="0.0" izz="0.0" ixy="-0.0" iyz="-0.0" ixz="-0.0"/>
+    <inertia ixx="0.001" iyy="0.0" izz="0.0" ixy="0.0" iyz="0.0" ixz="0.0"/>
   </inertial>
   <visual>
